Commit message: Update joint origins to remove z-offset

File: test_urdf/urdf/basic_robot.urdf (robot description, URDF)
Before this commit: robot deposition_robot, 11 links, 10 joints
Joints:
- joint base_to_deposition_joint: origin xyz=-0.22 0 0.075 rpy=0 0 0 -> xyz=-0.22 0 0.0 rpy=0 0 0
- joint base_to_extraction_joint: origin xyz=0.22 0 0.075 rpy=0 0 0 -> xyz=0.22 0 0.0 rpy=0 0 0
- joint front_right_steering_joint: origin xyz=0.32 -0.24 -0.075 rpy=0 0 0 -> xyz=0.32 -0.24 -0.0 rpy=0 0 0
- joint rear_left_steering_joint: origin xyz=-0.32 0.24 -0.075 rpy=0 0 0 -> xyz=-0.32 0.24 -0.0 rpy=0 0 0
- joint rear_right_steering_joint: origin xyz=-0.32 -0.24 -0.075 rpy=0 0 0 -> xyz=-0.32 -0.24 -0.0 rpy=0 0 0
