Commit message: updated urdf

File: src/description/urdf/basic_robot.urdf (robot description, URDF)
Before this commit: robot deposition_robot, 11 links, 10 joints
Joints:
- joint front_left_steering_joint: limit lower=-1.5708 upper=1.5708 effort=20.0 velocity=2.0 -> lower=-6.28 upper=6.28 effort=20.0 velocity=2.0; origin xyz=0.32 0.24 -0.075 rpy=0 0 0 -> xyz=0.32 0.24 -0.0 rpy=0 0 0
- joint front_right_steering_joint: limit lower=-1.5708 upper=1.5708 effort=20.0 velocity=2.0 -> lower=-6.28 upper=6.28 effort=20.0 velocity=2.0
- joint rear_left_steering_joint: limit lower=-1.5708 upper=1.5708 effort=20.0 velocity=2.0 -> lower=-6.28 upper=6.28 effort=20.0 velocity=2.0
- joint rear_right_steering_joint: limit lower=-1.5708 upper=1.5708 effort=20.0 velocity=2.0 -> lower=-6.28 upper=6.28 effort=20.0 velocity=2.0

Commit message: works, changed the pid of gazebo, tune tolerance

File: src/description/urdf/basic_robot.urdf (robot description, URDF)
Before this commit: robot deposition_robot, 11 links, 10 joints
Joints:
- joint front_left_steering_joint: limit lower=-6.28 upper=6.28 effort=20.0 velocity=2.0 -> lower=-6.28 upper=6.28 effort=100.0 velocity=2.0
- joint front_right_steering_joint: limit lower=-6.28 upper=6.28 effort=20.0 velocity=2.0 -> lower=-6.28 upper=6.28 effort=100.0 velocity=2.0

Commit message: added imu and camera

File: src/description/urdf/basic_robot.urdf (robot description, URDF)
Before this commit: robot deposition_robot, 11 links, 10 joints
Links:
- added link chassis, mass 68.0; collision box size=0.75 0.75 0.04; visual box size=0.75 0.75 0.04
- added link imu_link, mass 0.1
- added link top_camera_holder_link, mass 0.2; visual cylinder length=0.04 radius=0.04
- link base_link: mass 68.0 -> None; geometry 
- link extraction_system_link: geometry collision box size=0.40 0.30 0.34; visual box size=0.40 0.30 0.34
Joints:
- added joint chassis_joint: type fixed, parent base_link, child chassis, origin xyz=0 0 0.31 rpy=0 0 0
- added joint imu_joint: type fixed, parent chassis, child imu_link, origin xyz=0 0 0 rpy=0 0 0
- added joint top_camera_holder_joint: type continuous, parent chassis, child top_camera_holder_link, origin xyz=0.36 0 0.45 rpy=0 0 0, axis 0 0 1
- joint base_to_deposition_joint: parent base_link -> chassis
- joint base_to_extraction_joint: origin xyz=0.22 0 0.0 rpy=0 0 0 -> xyz=0.175 0 0.0 rpy=0 0 0; parent base_link -> chassis
- joint front_left_steering_joint: parent base_link -> chassis
- joint front_right_steering_joint: parent base_link -> chassis
- joint rear_left_steering_joint: parent base_link -> chassis
- joint rear_right_steering_joint: parent base_link -> chassis

Commit message: Limit update to standalone robot URDF

File: src/description/urdf/basic_robot.urdf (robot description, URDF)
Before this commit: robot melbot, 14 links, 13 joints
Links:
- added link front_camera_link, mass 0.072; collision box size=0.025 0.09 0.025; visual box size=0.025 0.09 0.025
- added link front_camera_optical_link
- added link top_camera_link, mass 0.072; collision box size=0.025 0.09 0.025; visual box size=0.025 0.09 0.025
- added link top_camera_optical_link
Joints:
- added joint front_camera_joint: type fixed, parent chassis, child front_camera_link, origin xyz=0.36 0 0.39 rpy=0 0.7853981633974483 0
- added joint front_camera_optical_joint: type fixed, parent front_camera_link, child front_camera_optical_link, origin xyz=0 0 0 rpy=-1.5707963267948966 0 -1.5707963267948966
- added joint top_camera_joint: type fixed, parent top_camera_holder_link, child top_camera_link, origin xyz=0.03 0 0.04 rpy=0 0 0
- added joint top_camera_optical_joint: type fixed, parent top_camera_link, child top_camera_optical_link, origin xyz=0 0 0 rpy=-1.5707963267948966 0 -1.5707963267948966

Commit message: Restore urdf to October 17 Melbot version

File: src/description/urdf/basic_robot.urdf (robot description, URDF)
Before this commit: robot melbot, 18 links, 17 joints
Links:
- removed link front_camera_link
- removed link front_camera_optical_link
- removed link top_camera_link
- removed link top_camera_optical_link
Joints:
- removed joint front_camera_joint
- removed joint front_camera_optical_joint
- removed joint top_camera_joint
- removed joint top_camera_optical_joint
